File: hardware/PCB_Prototipo/PCB_Prototipo.kicad_sch (KiCad schematic)
At the start: 0 parts

Commit message: Agregado el informe de planificación
Other:
- sheet Sensors_sheet renamed Top_Sensors_sheet
- added sheet Bottom_Sensors (Bottom_sensors.kicad_sch)
Changed lines of the file:
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@@
 			(color 0 0 0 0.0000)
 		)
-		(property "Sheetname" "Sensors_sheet"
+		(property "Sheetname" "Top_Sensors_sheet"
 			(at 22.86 17.0684 0)
 			(effects
@@
 				)
 			)
+		)
+	)
+	(sheet
+		(at 68.58 17.78)
+		(size 22.86 26.67)
+		(exclude_from_sim no)
+		(in_bom yes)
+		(on_board yes)
+		(dnp no)
+		(fields_autoplaced yes)
+		(stroke
+			(width 0.1524)
+			(type solid)
+		)
+		(fill
+			(color 0 0 0 0.0000)
+		)
+		(property "Sheetname" "Bottom_Sensors"
+			(at 68.58 17.0684 0)
+			(effects
+				(font
+					(size 1.27 1.27)
+				)
+				(justify left bottom)
+			)
+		)
+		(property "Sheetfile" "Bottom_sensors.kicad_sch"
+			(at 68.58 45.0346 0)
+			(effects
+				(font
+					(size 1.27 1.27)
+				)
+				(justify left top)
+			)
+		)
+		(instances
+			(project "PCB_Prototipo"
+				(path "/e94a28e3-abd7-45ed-8e41-e334e139ce43"
+					(page "3")
+				)
+			)
